Commit message: Merged remote main into local after pull

File: src/two_dof_robot/urdf/robot.urdf.xacro (robot description, xacro)
@@ -9,5 +9,5 @@
     <origin xyz="0 0 0.5" rpy="0 0 0"/>
     <axis xyz="0 0 1"/>
-    <limit lower="-1.57" upper="1.57" effort="1.0" velocity="1.0"/>
+    <limit lower="-3.14" upper="3.14" effort="1.0" velocity="1.0"/>
   </joint>
   <!-- Link 1 -->
@@ -25,5 +25,5 @@
     <child link="link2"/>
     <origin xyz="0 0.05 0.525" rpy="0 1.5708 0"/>
-    <axis xyz="0 1 0"/>
+    <axis xyz="0 0 1"/>
     <limit lower="-1.57" upper="1.57" effort="1.0" velocity="1.0"/>
   </joint>
@@ -31,7 +31,7 @@
   <link name="link2">
     <visual>
-      <origin xyz="0.05 0 0.5" rpy="0 0 0"/>
+      <origin xyz="0.05 -0.45 0.05" rpy="0 0 1.5708"/>
       <geometry>
-        <box size="0.05 0.05 1.05"/>
+        <box size="1.05 0.05 0.05"/>
       </geometry>
       <material name="green">
@@ -44,10 +44,10 @@
     <parent link="link2"/>
     <child link="end_effector"/>
-    <origin xyz="0 0 0.525" rpy="0 0 0"/> <!-- link2 yüksekliği/2 -->
+    <origin xyz="0 0 0" rpy="0 0 0"/> <!-- link2 yüksekliği/2 -->
   </joint>
   <!-- End Effector Link -->
   <link name="end_effector">
     <visual>
-      <origin xyz="0.05 0.0 0.5" rpy="0 0 0"/>
+      <origin xyz="0.05 -1.0 0.05" rpy="0 0 0"/>
       <geometry>
         <sphere radius="0.03"/>
